Commit message: fix : packagename

File: agv_amr/urdf/agv_amr.urdf (robot description, URDF)
Before this commit: robot sendbooster_amr, 4 links, 3 joints
Links:
- link base_link: geometry collision mesh filename=package://agv_amr/urdf/meshes/base_link.STL; visual mesh filename=package://agv_amr/urdf/meshes/base_link.STL
- link left_wheel: geometry collision mesh filename=package://agv_amr/urdf/meshes/left_wheel.STL; visual mesh filename=package://agv_amr/urdf/meshes/left_wheel.STL
- link right_wheel: geometry collision mesh filename=package://agv_amr/urdf/meshes/right_wheel.STL; visual mesh filename=package://agv_amr/urdf/meshes/right_wheel.STL
